File: PLS8_M2_Key_B_3042.kicad_sch (KiCad schematic)
At the start: 39 parts, among them Q2 2SK3018, Q3 2SK3018, Q4 2SK3018, U20 PLS8-E, U28 M2_KEYB_JSZ

Commit message: Use KiCad's built-in library for various symbols and footprints
Make general improvements to the legibility of the schematic.
Reuse some of the footprints from the dvk-mx8m-bsb project and others.
Redefine all pins which were left as "passive" to being their
corresponding functional definition.
Make sure the schematic is passing ERC (no errors or warnings).
Parts:
- removed ANT2, ANT3: IPEX20369, APEX-4, symbol PLS8_M2_Key_B_3042:3_mirrored_IPEX20369
- removed C1, C11, C2, C3, C335, C336, C5, C6, C7: C0402, CAP-0402, symbol PLS8_M2_Key_B_3042:0_C0402
- removed C10, C281, C283, C290, C299, C306, C329, C330, C4, C9: C0603, CAP-0603, symbol PLS8_M2_Key_B_3042:0_C0603
- removed C8: C0402, CAP-0402, symbol PLS8_M2_Key_B_3042:1_C0402
- removed L1, L11: BEAD-0402, IND-0402, symbol PLS8_M2_Key_B_3042:1_mirrored_BEAD-0402
- removed Q2, Q3, Q4: 2SK3018, DTC123JUA, symbol PLS8_M2_Key_B_3042:0_2SK3018
- removed R1, R3, R4: RES_2, RES-0402, symbol PLS8_M2_Key_B_3042:2_RES_2
- removed R133: RES_2, RES-0402, symbol PLS8_M2_Key_B_3042:0_RES_2
- removed R2, R223: RES_2, RES-0402, symbol PLS8_M2_Key_B_3042:1_RES_2
- removed R5: RES_2, RES-0402, symbol PLS8_M2_Key_B_3042:3_RES_2
- removed TP1, TP39: T_POINT_R, SIP-1PF, symbol PLS8_M2_Key_B_3042:3_mirrored_T_POINT_R
- removed TS4: SC-M2, SC-M4, symbol PLS8_M2_Key_B_3042:0_SC-M2
- added ANT2, ANT3: MHF4, PLS8_M2_Key_B_3042:MHF4_20449-001E, symbol Connector:Conn_Coaxial
- added C1, C11, C2, C3: 18pF, Capacitor_SMD:C_0402_1005Metric, symbol Device:C
- added C10, C281, C283, C290, C299, C306, C329, C330, C4, C7, C9: 22uF, Capacitor_SMD:C_0603_1608Metric, symbol Device:C
- added C335, C5, C8: 220nF, Capacitor_SMD:C_0402_1005Metric, symbol Device:C
- added C336, C6: 10nF, Capacitor_SMD:C_0402_1005Metric, symbol Device:C
- added L1, L11: 22nH, Inductor_SMD:L_0402_1005Metric, symbol Device:L
- added Q2, Q4: DMN61D9UWQ-13, Package_TO_SOT_SMD:SOT-323_SC-70, symbol PLS8_M2_Key_B_3042:DMN61D9UWQ-13
- added Q3: NC, Package_TO_SOT_SMD:SOT-323_SC-70, symbol PLS8_M2_Key_B_3042:DMN61D9UWQ-13
- added R1, R133, R3, R4: NC, Resistor_SMD:R_0402_1005Metric, symbol Device:R
- added R2, R5: 100, Resistor_SMD:R_0402_1005Metric, symbol Device:R
- added R223: 1k, Resistor_SMD:R_0402_1005Metric, symbol Device:R
- added TP1, TP39: TestPoint, PLS8_M2_Key_B_3042:TEST_POINT, symbol Connector:TestPoint
- added TS4: MountingHole_Pad, PLS8_M2_Key_B_3042:M.2_Mounting_Hole, symbol Mechanical:MountingHole_Pad
- added unit 2 of U20
- U20: value PLS8-E -> PLS8; footprint PLS8-E -> PLS8_M2_Key_B_3042:PLS8; symbol PLS8_M2_Key_B_3042:0_PLS8-E -> PLS8_M2_Key_B_3042:PLS8; DESCRIPTION Module Wireless 4G PLS8-E -> (none); DISPLAY_VALUE PLS8-E -> (none); Distrib Link (none) -> https://www.digikey.com/en/products/detail/thales-dis-forme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; Distrib PN (none) -> 2213-L30960-N3410-A400CT-ND; GEOMETRY.HEIGHT 2.5MM -> (none); MFG Name (none) -> Thales DIS; MFG Part Num (none) -> PLS8-US Rel.4; MFG_NAME Gemalto -> (none); Others (none) -> https://www.digikey.com/en/products/detail/thales-dis-forme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; PCB DECAL PLS8-E -> (none); PCB FOOTPRINT LGA -> (none); Tolerance (none) -> -
- U28: value M2_KEYB_JSZ -> M2_KEYB; footprint M2_KEYB_3042 -> PLS8_M2_Key_B_3042:M2_KEYB_3042; symbol PLS8_M2_Key_B_3042:0_M2_KEYB_JSZ -> PLS8_M2_Key_B_3042:M2_KEYB; PCB DECAL M2_KEYB_3042 -> (none)
Connections:
- net 4G_RESET: now also R5.1
- net CC_DET: now also Q2.3 (S)
- net GND: now also ANT2.2 (Ext), ANT3.2 (Ext), C10.2, C281.2, C283.2, C290.2, C299.2, C306.2, C329.2, C330.2, C335.1, C336.2, C4.2, C5.2, C6.2, C7.2, C8.2, C9.2, L1.1, L11.1, Q2.2 (D), Q3.2 (D), Q4.2 (D), R1.2, TS4.1; no longer U20.P4 (USB_DP), U20.P5 (USB_DN), U28.7 (USB_D+), U28.9 (USB_D-)
- net VBAT: now also C10.1, C281.1, C283.1, C290.1, C299.1, C306.1, C329.1, C4.1, C5.1, C6.1, C7.1, C9.1, R223.1; no longer U20.K14 (CCIO1), U20.K15 (CCVCC1), U20.L14 (CCRST1), U20.L15 (CCCLK1), U20.M10 (DOUT), U20.M7 (DIN), U20.M8 (BCLK), U20.M9 (FSC), U28.20 (PCM_CLK), U28.22 (PCM_IN), U28.24 (PCM_OUT), U28.28 (PCM_SYNC), U28.30 (UIM-RESET_(I)), U28.32 (UIM-CLK_(I)), U28.34 (UIM-DATA_(IO)), U28.36 (UIM-PWR_(I)), U28.6 (POWER_OFF(1_8V))
- net VEXT_1V8: now also R133.1
- net WOWWAN: now also R2.1
- net at U20.A12 (ANT_DRX_MIMO): now also C2.2
- net at U20.K1 (ANT_MAIN): now also C3.2
- net at U20.L16 (IGT): now also Q4.3 (S), R1.1, R4.2
- net at U20.M15 (VDDLP): now also C330.1
- net at U20.N14 (EMERG_OFF): now also Q3.3 (S)
- net at U20.N5 (VUSB_IN): now also C8.1, R223.2
- net at U20.P10 (RING0): now also R2.2
- net at U20.P11 (RXD0): now also TP1.1
- net at U20.P12 (TXD0): now also TP39.1
- net at U28.66 (SIM_DETECT_(O)): now also Q2.1 (GATE), R133.2
- new net: Q4.1 (GATE), R3.2, R4.1, R5.2
- new net: ANT3.1 (In), C11.1
- new net: C11.2, C3.1, L11.2
- new net: C1.2, C2.1, L1.2
- new net: ANT2.1 (In), C1.1
- new net 4G_ON/OFF: Q3.1 (GATE), R3.1, U28.6 (POWER_OFF(1_8V))
- new net CCCLK: U20.L15 (CCCLK1), U28.32 (UIM-CLK_(I))
- new net CCIO: U20.K14 (CCIO1), U28.34 (UIM-DATA_(IO))
- new net CCRST: C336.1, U20.L14 (CCRST1), U28.30 (UIM-RESET_(I))
- new net CCVCC: C335.2, U20.K15 (CCVCC1), U28.36 (UIM-PWR_(I))
- new net PCM_BCLK: U20.M8 (BCLK), U28.20 (PCM_CLK)
- new net PCM_DIN: U20.M7 (DIN), U28.22 (PCM_IN)
- new net PCM_DOUT: U20.M10 (DOUT), U28.24 (PCM_OUT)
- new net PCM_SYNC: U20.M9 (FSC), U28.28 (PCM_SYNC)
- new net USB_DN: U20.P5 (USB_DN), U28.9 (USB_D-)
- new net USB_DP: U20.P4 (USB_DP), U28.7 (USB_D+)
- no-connect marks 0 -> 105
Other:
- note removed: "1"
- note removed: "A"
- note removed: "Date:"
- note removed: "Design by:"
- note removed: "Drawing Title:"
- note removed: "PLS8 M.2 Key B 3042"
- note removed: "PSL8_M2_Key_B_3042"
- note removed: "Page Title:"
- note removed: "Purism"
- note removed: "Rev:"
- note removed: "Sheet"
- note removed: "of"
- note removed: "v0.5.0"
- title: (none) -> PLS8 M.2 Key B 3042 WWAN Module
- moved on the sheet: U28

Commit message: Update the footprints in the layout using the ones assigned in the previous commit
Make C7 10nF as it was previously.
Fix the copper pour settings to make sure all connections are properly
made.
Adjust ATN2 and ANT3's footprint to have an underlying pad which copper
pour can connect to.
Parts:
- C7: value 22uF -> 10nF; footprint Capacitor_SMD:C_0603_1608Metric -> Capacitor_SMD:C_0402_1005Metric; Distrib Link https://www.digikey.com/en/products/detail/samsung-electro-mechanics/CL10A226MP8NUNE/3886932 -> https://www.digikey.com/en/products/detail/samsung-electro-mechanics/CL05B103KB5NNNC/3886686; Distrib PN 1276-1274-1-ND -> 1276-1028-1-ND; MFG Part Num CL10A226MP8NUNE -> CL05B103KB5NNNC; Others https://www.digikey.com/en/products/filter/ceramic-capacitors/60?s=N4IgjCBcpgbFoDGUBmBDANgZwKYBoQB7KAbRAGYBOAJgBZ4BdAgBwBcoQBlVgJwEsAdgHMQAXwJhKADkoIQySOmz4ipEAAYQTEGw7d%2BwsQWrras6PNSZcBYpDLVqAAgCtAMS0t2kEAFUBfKwA8igAsjhoWACuPDhioqJAA -> https://www.digikey.com/en/products/filter/ceramic-capacitors/60?s=N4IgjCBcpgLFoDGUBmBDANgZwKYBoQB7KAbXAFYBOAJlgHYQCxLYAOWeA6gZlbt8YgAbJSHVKIALoEADgBcoIAMpyATgEsAdgHMQAXyZCEIZJHTZ8RUiG6Uw5VlNkLIytVt0HwlVhOgnUTFwCYkgyAAYnEHlFFQ0dfS5w2D8kQIsQ6zBwnPCAAhkAMSiY1wBVTXU5AHkUAFkcNCwAV1UcfT09IA; Tolerance 20% -> 10%
Connections:
- no-connect marks 105 -> 97
Other:
- moved on the sheet: ANT2, ANT3, C1, C10, C11, C2, C281, C283, C290, C299, C3, C306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
